File: unicorn/unicorn.kicad_sch (KiCad schematic)
At the start: 25 parts, among them J0 Conn_01x02, J1 Conn_01x14_Female, J2 Conn_01x14_Female, J3 SPI, U1 ATmega328-P, U2 L7805

Commit message: Unicorn - Feat/fix components (#2)
* replace power connector
- still need to redo routing

* fix routing + replace power connector with the right one

* add jst connector + update step file
Parts:
- J0: footprint Connector_JST:JST_PH_S2B-PH-K_1x02_P2.00mm_Horizontal -> JST_S2B-PH-SM4-TB:JST_S2B-PH-SM4-TB
- LED3: value Tx -> TX
- LED4: value Rx -> RX
Changed lines of the file:
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@@
     (title "Unicorn")
     (date "2023-08-03")
-    (rev "A")
+    (rev "B")
     (comment 1 "Author: Simone Girardi")
   )
@@
       (effects (font (size 1.27 1.27)))
     )
-    (property "Value" "Rx" (at 263.8425 43.18 0)
+    (property "Value" "RX" (at 263.8425 43.18 0)
       (effects (font (size 1.27 1.27)))
     )
@@
       (effects (font (size 1.27 1.27)) (justify left))
     )
-    (property "Footprint" "Connector_JST:JST_PH_S2B-PH-K_1x02_P2.00mm_Horizontal" (at 33.655 31.75 0)
+    (property "Footprint" "JST_S2B-PH-SM4-TB:JST_S2B-PH-SM4-TB" (at 33.655 31.75 0)
       (effects (font (size 1.27 1.27)) hide)
     )
@@
       (effects (font (size 1.27 1.27)))
     )
-    (property "Value" "Tx" (at 263.8425 33.02 0)
-      (effects (font (size 1.27 1.27)))
-    )
+    (property "Value" "TX" (at 263.8425 33.02 0)
+      (effects (font (size 1.27 1.27)))
+    )
