File: unicorn/kicad/unicorn.kicad_pcb (KiCad board)
At the start: 2 copper layers, 35 x 75 mm, 26 parts, among them J1 Conn_01x02, J2 SPI, J3 Conn_01x14_Female, J4 Conn_01x14_Female, U1 L7805, U2 ATmega328-P

Commit message: Add mounting holes
Routing:
- net Net-(J2-Pin_1): track 81.4 -> 87.5 mm
- net Net-(J1-Pin_1): track 43.4 -> 47.0 mm
Other:
- outline, holes or cut-outs redrawn
Changed lines of the file:
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@@
     (property "ki_keywords" "connector")
     (attr through_hole)
-    (fp_text reference "J2" (at 5.1816 2.3876 90) (layer "F.SilkS")
-        (effects (font (size 1 1) (thickness 0.15)))
-    )
-    (fp_text value "SPI" (at 1.27 7.41) (layer "F.Fab")
-        (effects (font (size 1 1) (thickness 0.15)))
-    )
-    (fp_text user "${REFERENCE}" (at 1.27 2.54 90) (layer "F.Fab")
+    (fp_text reference "J2" (at 5.1816 2.3876 90) (layer "F.SilkS") hide
+        (effects (font (size 1 1) (thickness 0.15)))
+    )
+    (fp_text value "SPI" (at -5.6388 2.1844) (layer "F.Fab") hide
         (effects (font (size 1 1) (thickness 0.15)))
     )
@@
         (effects (font (size 1 1) (thickness 0.15)))
     )
-    (fp_text value "100nF" (at 4.826 0) (layer "F.Fab")
+    (fp_text value "100nF" (at 0.8944 2.8864 90) (layer "F.Fab")
         (effects (font (size 1 1) (thickness 0.15)))
     )
@@
     (property "ki_keywords" "connector")
     (attr through_hole)
-    (fp_text reference "J4" (at 0 -2.77) (layer "F.SilkS")
-        (effects (font (size 1 1) (thickness 0.15)))
-    )
-    (fp_text value "Conn_01x14_Female" (at 0 35.79) (layer "F.Fab")
+    (fp_text reference "J4" (at 0 -2.77) (layer "F.SilkS") hide
+        (effects (font (size 1 1) (thickness 0.15)))
+    )
+    (fp_text value "Conn_01x14_Female" (at -3.0988 16.0782 90) (layer "F.Fab")
         (effects (font (size 1 1) (thickness 0.15)))
     )
@@
     (property "ki_keywords" "connector")
     (attr through_hole)
-    (fp_text reference "J3" (at -0.127 35.687) (layer "F.SilkS")
-        (effects (font (size 1 1) (thickness 0.15)))
-    )
-    (fp_text value "Conn_01x14_Female" (at 0 35.79) (layer "F.Fab")
+    (fp_text reference "J3" (at -0.127 35.687) (layer "F.SilkS") hide
+        (effects (font (size 1 1) (thickness 0.15)))
+    )
+    (fp_text value "Conn_01x14_Female" (at -3.556 17.4591 90) (layer "F.Fab")
         (effects (font (size 1 1) (thickness 0.15)))
     )
@@
         (effects (font (size 1 1) (thickness 0.15)))
     )
-    (fp_text value "100nF" (at 4.826 0.06) (layer "F.Fab")
+    (fp_text value "100nF" (at 1.0468 3.6576 90) (layer "F.Fab")
         (effects (font (size 1 1) (thickness 0.15)))
     )
@@
         (effects (font (size 1 1) (thickness 0.15)))
     )
-    (fp_text value "L7805" (at 7.985 4.135 90) (layer "F.Fab")
+    (fp_text value "L7805" (at -0.0508 4.0894 90) (layer "F.Fab")
         (effects (font (size 1 1) (thickness 0.15)))
     )
@@
         (effects (font (size 1 1) (thickness 0.15)))
     )
-    (fp_text value "10uF" (at 1 3.75 90) (layer "F.Fab") hide
+    (fp_text value "10uF" (at 1 3.75 90) (layer "F.Fab")
         (effects (font (size 1 1) (thickness 0.15)))
     )
@@
         (effects (font (size 1 1) (thickness 0.15)))
     )
-    (fp_text value "100uF" (at 4.515112 -0.14) (layer "F.Fab")
+    (fp_text value "100uF" (at 1 -2.5 90) (layer "F.Fab")
         (effects (font (size 1 1) (thickness 0.15)))
     )
@@
   (gr_line (start 159.75 134) (end 159.75 61)
     (stroke (width 0.1) (type solid)) (layer "Edge.Cuts"))
+  (gr_circle (center 158.2479 133.5) (end 159.2479 133.5)
+    (stroke (width 0.1) (type default)) (fill none) (layer "Edge.Cuts"))
+  (gr_circle (center 142.2525 71.0184) (end 143.2525 71.0184)
+    (stroke (width 0.1) (type default)) (fill none) (layer "Edge.Cuts"))
   (gr_line (start 124.75 61) (end 124.75 134)
     (stroke (width 0.1) (type solid)) (layer "Edge.Cuts"))
@@
   (gr_arc (start 159.75 134) (mid 159.479108 134.68523) (end 158.812893 135)
     (stroke (width 0.1) (type solid)) (layer "Edge.Cuts"))
+  (gr_circle (center 126.2519 133.5) (end 127.2519 133.5)
+    (stroke (width 0.1) (type default)) (fill none) (layer "Edge.Cuts"))
   (gr_text "Unicorn rev_B" (at 142.2525 114.7125 90) (layer "B.SilkS")
     (effects (font (size 2 2) (thickness 0.2)) (justify mirror))
@@
     (format (prefix "") (suffix "") (units 3) (units_format 1) (precision 4))
     (style (thickness 0.15) (arrow_length 1.27) (text_position_mode 0) (extension_height 0.58642) (extension_offset 0.5) keep_text_aligned)
+  )
+  (dimension (type radial) (layer "Eco1.User")
+    (pts (xy 158.2479 133.5) (xy 158.2479 132.5))
+    (leader_length 2.318048)
+    (gr_text "R 1.000 mm" (at 164.6936 130.181952) (layer "Eco1.User")
+      (effects (font (size 1 1) (thickness 0.15)))
+    )
+    (format (prefix "R ") (suffix "") (units 3) (units_format 1) (precision 3))
+    (style (thickness 0.15) (arrow_length 1.27) (text_position_mode 0) (extension_offset 0.5) keep_text_aligned)
   )
   (segment (start 129.54 79.93) (end 129.54 85.8) (width 0.3) (layer "F.Cu") (net 1))
@@
   (segment (start 151.049 77.708) (end 151.049 81.849) (width 0.3) (layer "F.Cu") (net 4))
   (segment (start 129.54 74.64) (end 131.155 73.025) (width 0.3) (layer "B.Cu") (net 4))
-  (segment (start 146.151 73.025) (end 155 81.8743) (width 0.3) (layer "B.Cu") (net 4))
-  (segment (start 131.155 73.025) (end 146.151 73.025) (width 0.3) (layer "B.Cu") (net 4))
-  (segment (start 155 81.8743) (end 155 85.8) (width 0.3) (layer "B.Cu") (net 4))
-  (segment (start 132.842 123.952) (end 132.842 67.51) (width 0.3) (layer "F.Cu") (net 5))
-  (segment (start 132.842 67.51) (end 131.142 65.81) (width 0.3) (layer "F.Cu") (net 5))
-  (segment (start 141.732 124.841) (end 133.731 124.841) (width 0.3) (layer "F.Cu") (net 5))
-  (segment (start 133.731 124.841) (end 132.842 123.952) (width 0.3) (layer "F.Cu") (net 5))
+  (segment (start 155 75.8028) (end 155 85.8) (width 0.3) (layer "B.Cu") (net 4))
+  (segment (start 131.155 73.025) (end 152.2222 73.025) (width 0.3) (layer "B.Cu") (net 4))
+  (segment (start 152.2222 73.025) (end 155 75.8028) (width 0.3) (layer "B.Cu") (net 4))
   (segment (start 146.0725 126.1525) (end 143.0435 126.1525) (width 0.3) (layer "F.Cu") (net 5))
   (segment (start 143.0435 126.1525) (end 141.732 124.841) (width 0.3) (layer "F.Cu") (net 5))
+  (segment (start 133.731 124.841) (end 132.6388 123.7488) (width 0.3) (layer "F.Cu") (net 5))
+  (segment (start 141.732 124.841) (end 133.731 124.841) (width 0.3) (layer "F.Cu") (net 5))
+  (segment (start 132.6388 67.3068) (end 131.142 65.81) (width 0.3) (layer "F.Cu") (net 5))
+  (segment (start 132.6388 123.7488) (end 132.6388 67.3068) (width 0.3) (layer "F.Cu") (net 5))
   (segment (start 146.073 126.152) (end 146.0725 126.1525) (width 0.3) (layer "B.Cu") (net 5))
   (segment (start 154.9205 126.152) (end 146.073 126.152) (width 0.3) (layer "B.Cu") (net 5))
@@
   (segment (start 154.94 118.5125) (end 146.0925 118.5125) (width 0.3) (layer "B.Cu") (net 13))
   (segment (start 146.0925 118.5125) (end 146.0725 118.5325) (width 0.3) (layer "B.Cu") (net 13))
-  (segment (start 129.286 61.595) (end 131.953 61.595) (width 0.3) (layer "F.Cu") (net 14))
-  (segment (start 140.97 70.612) (end 140.97 118.491) (width 0.3) (layer "F.Cu") (net 14))
-  (segment (start 140.97 118.491) (end 146.0725 123.5935) (width 0.3) (layer "F.Cu") (net 14))
+  (segment (start 131.953 61.595) (end 129.286 61.595) (width 0.3) (layer "F.Cu") (net 14))
+  (segment (start 144.7864 122.3264) (end 134.366 122.3264) (width 0.3) (layer "F.Cu") (net 14))
+  (segment (start 133.1888 121.1492) (end 133.1888 62.8308) (width 0.3) (layer "F.Cu") (net 14))
+  (segment (start 133.1888 62.8308) (end 131.953 61.595) (width 0.3) (layer "F.Cu") (net 14))
+  (segment (start 134.366 122.3264) (end 133.1888 121.1492) (width 0.3) (layer "F.Cu") (net 14))
+  (segment (start 129.286 61.595) (end 128.602 62.279) (width 0.3) (layer "F.Cu") (net 14))
   (segment (start 146.0725 123.6125) (end 146.0915 123.6125) (width 0.3) (layer "F.Cu") (net 14))
-  (segment (start 131.953 61.595) (end 140.97 70.612) (width 0.3) (layer "F.Cu") (net 14))
+  (segment (start 146.0725 123.6125) (end 144.7864 122.3264) (width 0.3) (layer "F.Cu") (net 14))
+  (segment (start 128.602 62.279) (end 128.602 63.27) (width 0.3) (layer "F.Cu") (net 14))
   (segment (start 146.0725 123.5935) (end 146.0725 123.6125) (width 0.3) (layer "F.Cu") (net 14))
-  (segment (start 128.602 63.27) (end 128.602 62.279) (width 0.3) (layer "F.Cu") (net 14))
-  (segment (start 128.602 62.279) (end 129.286 61.595) (width 0.3) (layer "F.Cu") (net 14))
   (segment (start 146.073 123.612) (end 154.9205 123.612) (width 0.3) (layer "B.Cu") (net 14))
   (segment (start 146.072 123.612) (end 146.073 123.612) (width 0.3) (layer "B.Cu") (net 14))
